File: hardware/graphite.kicad_pcb (KiCad board)
At the start: 2 copper layers, 102 parts, among them J1 Adafruit TFT

Commit message: feat: finished routing :tada:
Parts:
- A1: moved to B.Cu
- D1: moved to F.Cu
- moved D41 156.8 mm to (78.7, 180.3), turned to 90 degrees
- moved D46 154.2 mm to (78.7, 193.0), turned to 90 degrees
- moved J1 147.9 mm to (91.4, 22.9)
- moved D42 143.1 mm to (92.7, 180.3), turned to 90 degrees
- moved D47 140.4 mm to (92.7, 193.0), turned to 90 degrees
- moved D31 131.0 mm to (78.7, 154.9), turned to 90 degrees
- moved D43 129.6 mm to (106.7, 180.3), turned to 90 degrees
- moved D36 129.3 mm to (78.7, 167.6), turned to 90 degrees
- moved D48 126.7 mm to (106.7, 193.0), turned to 90 degrees
- moved D27 117.7 mm to (92.7, 139.7), turned to 90 degrees
- moved D32 116.7 mm to (92.7, 154.9), turned to 90 degrees
- moved D44 116.2 mm to (120.7, 180.3), turned to 90 degrees
- moved D37 115.0 mm to (92.7, 167.6), turned to 90 degrees
- moved D49 113.2 mm to (120.7, 193.0), turned to 90 degrees
- moved D16 112.1 mm to (78.7, 110.5), turned to 90 degrees
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Routing:
- net ROW9: track 0.00 -> 240.1 mm
- net ROW8: track 0.00 -> 229.4 mm
- net ROW7: track 0.00 -> 221.4 mm
- net COL0: track 0.00 -> 215.4 mm
- net ROW6: track 0.00 -> 210.8 mm
- net ROW5: track 0.00 -> 197.5 mm
- net COL1: track 0.00 -> 197.4 mm
- net ROW4: track 0.00 -> 184.9 mm
- net COL2: track 0.00 -> 179.1 mm
- net COL3: track 0.00 -> 177.8 mm, vias 0 -> 2
- net ROW1: track 0.00 -> 176.4 mm
- net ROW3: track 0.00 -> 171.8 mm
- net ROW2: track 0.00 -> 157.7 mm
- net COL4: track 0.00 -> 147.9 mm, vias 0 -> 2
- net ROW0: track 0.00 -> 132.5 mm
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Other:
- board outline added: 86.4 x 177.8 mm
- board text added: "*rpi pico here*"
- board text added: "github.com/thelegendofmario/graphite"
- board text added: "graphite v1r1"
