File: hardware/graphite.kicad_sch (KiCad schematic)
At the start: 0 parts

Commit message: chore: hopefully actually wired screen correctly lol
Parts:
- added A1: RaspberryPi_Pico, Module_RaspberryPi_Pico:RaspberryPi_Pico_Common, symbol Rasberry_Pi_Pico:RaspberryPi_Pico
- added J1: Adafruit TFT, symbol Connector_Generic:Conn_01x10
- added S1: B3F-1000, B3F1002, symbol OmronB3F_1000:B3F-1000
Connections:
- new net +3V3: A1.36 (3V3), J1.9 (Pin_9)
- new net +5V: A1.40 (VBUS)
- new net BL: A1.22 (GPIO17), J1.1 (Pin_1)
- new net CS: A1.26 (GPIO20), J1.5 (Pin_5)
- new net D/C: A1.29 (GPIO22), J1.8 (Pin_8)
- new net GND: A1.13 (GND), A1.18 (GND), A1.23 (GND), A1.28 (GND), A1.3 (GND), A1.33 (AGND), A1.38 (GND), A1.8 (GND), J1.10 (Pin_10)
- new net MISO: A1.21 (GPIO16), J1.3 (Pin_3)
- new net MOSI: A1.25 (GPIO19), J1.4 (Pin_4)
- new net RST: A1.31 (GPIO26_ADC0), J1.7 (Pin_7)
- new net SCK: A1.24 (GPIO18), J1.2 (Pin_2)
- new net SDCS: A1.27 (GPIO21), J1.6 (Pin_6)
Other:
- note added: "BL SCK MISO MOSI CS SDCS RST D/C VIN GND"

Commit message: feat: finished schematic
Parts:
- added D1, D10, D11, D12, D13, D14, D15, D16, D17, D18, D19, D2, D20, D21, D22, D23, D24, D25, D26, D27, D28, D29, D3, D30, D31, D32, D33, D34, D35, D36, D37, D38, D39, D4, D40, D41, D42, D43, D44, D45, D46, D47, D48, D49, D5, D50, D6, D7, D8, D9: 1N4148, Diode_THT:D_DO-35_SOD27_P7.62mm_Horizontal, symbol Diode:1N4148
- added S10, S11, S12, S13, S14, S15, S16, S17, S18, S19, S2, S20, S21, S22, S23, S24, S25, S26, S27, S28, S29, S3, S30, S31, S32, S33, S34, S35, S36, S37, S38, S39, S4, S40, S41, S42, S43, S44, S45, S46, S47, S48, S49, S5, S50, S6, S7, S8, S9: B3F-1000, symbol OmronB3F_1000:B3F-1000
- S1: footprint B3F1002 -> (none)
Connections:
- net at S1.2: now also D2.2 (A)
- net COL1: now reaches S1.3
- net COL1: now also A1.2 (GPIO1), S13.3, S17.3, S22.3, S27.3, S32.3, S37.3, S42.3, S47.3, S6.3
- net COL0: now reaches A1.1 (GPIO0)
- net COL0: now also S11.3, S12.3, S16.3, S21.3, S26.3, S31.3, S36.3, S41.3, S46.3, S5.3
- net ROW1: now reaches A1.10 (GPIO7)
- net ROW1: now also D10.1 (K), D11.1 (K), D6.1 (K), D7.1 (K), D8.1 (K), D9.1 (K)
- net ROW2: now reaches A1.11 (GPIO8)
- net ROW2: now also D12.1 (K), D13.1 (K), D14.1 (K), D15.1 (K)
- net ROW3: now reaches A1.12 (GPIO9)
- net ROW3: now also D16.1 (K), D17.1 (K), D18.1 (K), D19.1 (K), D20.1 (K)
- net ROW4: now reaches A1.14 (GPIO10)
- net ROW4: now also D21.1 (K), D22.1 (K), D23.1 (K), D24.1 (K), D25.1 (K)
- net ROW5: now reaches A1.15 (GPIO11)
- net ROW5: now also D26.1 (K), D27.1 (K), D28.1 (K), D29.1 (K), D30.1 (K)
- net ROW6: now reaches A1.16 (GPIO12)
- net ROW6: now also D31.1 (K), D32.1 (K), D33.1 (K), D34.1 (K), D35.1 (K)
- net ROW7: now reaches A1.17 (GPIO13)
- net ROW7: now also D36.1 (K), D37.1 (K), D38.1 (K), D39.1 (K), D40.1 (K)
- net ROW8: now reaches A1.19 (GPIO14)
- net ROW8: now also D41.1 (K), D42.1 (K), D43.1 (K), D44.1 (K), D45.1 (K)
- net ROW9: now reaches A1.20 (GPIO15)
- net ROW9: now also D46.1 (K), D47.1 (K), D48.1 (K), D49.1 (K), D50.1 (K)
- net COL2: now reaches A1.4 (GPIO2)
- net COL2: now also S14.3, S18.3, S2.3, S23.3, S28.3, S33.3, S38.3, S43.3, S48.3, S7.3
- net COL3: now reaches A1.5 (GPIO3)
- net COL3: now also S15.3, S19.3, S24.3, S29.3, S3.3, S34.3, S39.3, S44.3, S49.3, S8.3
- net COL4: now reaches A1.6 (GPIO4)
- net COL4: now also S20.3, S25.3, S30.3, S35.3, S4.3, S40.3, S45.3, S50.3, S9.3
- net COL5: now reaches A1.7 (GPIO5)
- net COL5: now also S10.3
- net ROW0: now reaches A1.9 (GPIO6)
- net ROW0: now also D1.1 (K), D2.1 (K), D3.1 (K), D4.1 (K), D5.1 (K)
- new net: D11.2 (A), S10.2
- new net: D32.2 (A), S32.2
- new net: D26.2 (A), S26.2
- new net: D49.2 (A), S49.2
- new net: D40.2 (A), S40.2
- new net: D12.2 (A), S12.2
- new net: D34.2 (A), S34.2
- new net: D48.2 (A), S48.2
- new net: D30.2 (A), S30.2
- new net: D33.2 (A), S33.2
- new net: D35.2 (A), S35.2
- new net: D41.2 (A), S41.2
- new net: D28.2 (A), S28.2
- new net: D8.2 (A), S7.2
- new net: D9.2 (A), S8.2
- new net: D18.2 (A), S18.2
- new net: D36.2 (A), S36.2
- new net: D3.2 (A), S2.2
- new net: D25.2 (A), S25.2
- new net: D44.2 (A), S44.2
- new net: D43.2 (A), S43.2
- new net: D14.2 (A), S14.2
- new net: D5.2 (A), S4.2
- new net: D23.2 (A), S23.2
- new net: D6.2 (A), S5.2
- new net: D27.2 (A), S27.2
- new net: D21.2 (A), S21.2
- new net: D47.2 (A), S47.2
- new net: D31.2 (A), S31.2
- new net: D7.2 (A), S6.2
- new net: D20.2 (A), S20.2
- new net: D37.2 (A), S37.2
- new net: D1.2 (A), S11.2
- new net: D22.2 (A), S22.2
- new net: D10.2 (A), S9.2
- new net: D38.2 (A), S38.2
- new net: D24.2 (A), S24.2
- new net: D17.2 (A), S17.2
- new net: D19.2 (A), S19.2
- new net: D39.2 (A), S39.2
- new net: D16.2 (A), S16.2
- new net: D45.2 (A), S45.2
- new net: D46.2 (A), S46.2
- new net: D13.2 (A), S13.2
- new net: D15.2 (A), S15.2
- new net: D29.2 (A), S29.2
- new net: D50.2 (A), S50.2
- new net: D4.2 (A), S3.2
- new net: D42.2 (A), S42.2
Other:
- note removed: "BL SCK MISO MOSI CS SDCS RST D/C VIN GND"
- title: (none) -> Graphite
- moved on the sheet: A1, J1

Commit message: chore: tidied up schematic
Parts:
- A1: footprint Module_RaspberryPi_Pico:RaspberryPi_Pico_Common -> Module:RaspberryPi_Pico_Common_THT
- J1: footprint (none) -> Connector_PinHeader_2.54mm:PinHeader_1x10_P2.54mm_Vertical
- S1, S10, S11, S12, S13, S14, S15, S16, S17, S18, S19, S2, S20, S21, S22, S23, S24, S25, S26, S27, S28, S29, S3, S30, S31, S32, S33, S34, S35, S36, S37, S38, S39, S4, S40, S41, S42, S43, S44, S45, S46, S47, S48, S49, S5, S50, S6, S7, S8, S9: footprint (none) -> B3F_1000:B3F1002
Changed lines of the file:
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@@
 			)
 		)
-		(property "Footprint" ""
+		(property "Footprint" "B3F_1000:B3F1002"
 			(at 220.98 155.88 0)
 			(effects
@@
 			)
 		)
-		(property "Footprint" ""
+		(property "Footprint" "B3F_1000:B3F1002"
 			(at 107.95 258.75 0)
 			(effects
@@
 			)
 		)
-		(property "Footprint" ""
+		(property "Footprint" "B3F_1000:B3F1002"
 			(at 78.74 237.16 0)
 			(effects
@@
 			)
 		)
-		(property "Footprint" ""
+		(property "Footprint" "B3F_1000:B3F1002"
 			(at 193.04 279.07 0)
 			(effects
@@
 			)
 		)
-		(property "Footprint" ""
+		(property "Footprint" "B3F_1000:B3F1002"
 			(at 78.74 176.2 0)
 			(effects
@@
 			)
 		)
-		(property "Footprint" ""
+		(property "Footprint" "B3F_1000:B3F1002"
 			(at 193.04 237.16 0)
 			(effects
@@
 			)
 		)
-		(property "Footprint" ""
+		(property "Footprint" "B3F_1000:B3F1002"
 			(at 137.16 258.75 0)
 			(effects
@@
 			)
 		)
-		(property "Footprint" ""
+		(property "Footprint" "B3F_1000:B3F1002"
 			(at 193.04 258.75 0)
 			(effects
@@
 			)
 		)
-		(property "Footprint" ""
+		(property "Footprint" "B3F_1000:B3F1002"
 			(at 107.95 135.56 0)
 			(effects
@@
 			)
 		)
-		(property "Footprint" ""
+		(property "Footprint" "B3F_1000:B3F1002"
 			(at 137.16 237.16 0)
 			(effects
@@
 			)
 		)
-		(property "Footprint" ""
+		(property "Footprint" "B3F_1000:B3F1002"
 			(at 165.1 155.88 0)
 			(effects
@@
 			)
 		)
-		(property "Footprint" ""
+		(property "Footprint" "B3F_1000:B3F1002"
 			(at 137.16 196.52 0)
 			(effects
@@
 			)
 		)
-		(property "Footprint" ""
+		(property "Footprint" "B3F_1000:B3F1002"
 			(at 165.1 299.39 0)
 			(effects
@@
 			)
 		)
-		(property "Footprint" ""
+		(property "Footprint" "B3F_1000:B3F1002"
 			(at 137.16 299.39 0)
 			(effects
@@
 			)
 		)
-		(property "Footprint" ""
+		(property "Footprint" "B3F_1000:B3F1002"
 			(at 137.16 176.2 0)
 			(effects
@@
 			)
 		)
-		(property "Footprint" ""
+		(property "Footprint" "B3F_1000:B3F1002"
 			(at 137.16 216.84 0)
 			(effects
@@
 			)
 		)
-		(property "Footprint" ""
+		(property "Footprint" "B3F_1000:B3F1002"
 			(at 107.95 237.16 0)
 			(effects
@@
 			)
 		)
-		(property "Footprint" ""
+		(property "Footprint" "B3F_1000:B3F1002"
 			(at 78.74 216.84 0)
 			(effects
@@
 			)
 		)
-		(property "Footprint" ""
+		(property "Footprint" "B3F_1000:B3F1002"
 			(at 78.74 258.75 0)
 			(effects
@@
 			)
 		)
-		(property "Footprint" ""
+		(property "Footprint" "B3F_1000:B3F1002"
 			(at 78.74 279.07 0)
 			(effects
@@
 			)
 		)
-		(property "Footprint" "Module_RaspberryPi_Pico:RaspberryPi_Pico_Common"
+		(property "Footprint" "Module:RaspberryPi_Pico_Common_THT"
 			(at 278.13 156.21 0)
 			(effects
@@
 			)
 		)
-		(property "Footprint" ""
+		(property "Footprint" "B3F_1000:B3F1002"
 			(at 165.1 258.75 0)
 			(effects
@@
 			)
 		)
-		(property "Footprint" ""
+		(property "Footprint" "B3F_1000:B3F1002"
 			(at 107.95 279.07 0)
 			(effects
@@
 			)
 		)
-		(property "Footprint" ""
+		(property "Footprint" "B3F_1000:B3F1002"
 			(at 193.04 155.88 0)
 			(effects
@@
 			)
 		)
-		(property "Footprint" ""
+		(property "Footprint" "Connector_PinHeader_2.54mm:PinHeader_1x10_P2.54mm_Vertical"
 			(at 340.36 113.03 0)
 			(effects
@@
 			)
 		)
-		(property "Footprint" ""
+		(property "Footprint" "B3F_1000:B3F1002"
 			(at 78.74 155.88 0)
 			(effects
@@
 			)
 		)
-		(property "Footprint" ""
+		(property "Footprint" "B3F_1000:B3F1002"
 			(at 137.16 135.56 0)
 			(effects
@@
 			)
 		)
-		(property "Footprint" ""
+		(property "Footprint" "B3F_1000:B3F1002"
 			(at 165.1 279.07 0)
 			(effects
@@
 			)
 		)
-		(property "Footprint" ""
+		(property "Footprint" "B3F_1000:B3F1002"
 			(at 165.1 216.84 0)
 			(effects
@@
 			)
 		)
-		(property "Footprint" ""
+		(property "Footprint" "B3F_1000:B3F1002"
 			(at 78.74 319.71 0)
 			(effects
@@
 			)
 		)
-		(property "Footprint" ""
+		(property "Footprint" "B3F_1000:B3F1002"
 			(at 137.16 319.71 0)
 			(effects
@@
 			)
 		)
-		(property "Footprint" ""
+		(property "Footprint" "B3F_1000:B3F1002"
 			(at 137.16 279.07 0)
 			(effects
@@
 			)
 		)
-		(property "Footprint" ""
+		(property "Footprint" "B3F_1000:B3F1002"
 			(at 165.1 176.2 0)
 			(effects
@@
 			)
 		)
-		(property "Footprint" ""
+		(property "Footprint" "B3F_1000:B3F1002"
 			(at 107.95 176.2 0)
 			(effects
@@
 			)
 		)
-		(property "Footprint" ""
+		(property "Footprint" "B3F_1000:B3F1002"
 			(at 78.74 135.56 0)
 			(effects
@@
 			)
 		)
-		(property "Footprint" ""
+		(property "Footprint" "B3F_1000:B3F1002"
 			(at 165.1 237.16 0)
 			(effects
@@
 			)
 		)
-		(property "Footprint" ""
+		(property "Footprint" "B3F_1000:B3F1002"
 			(at 137.16 155.88 0)
 			(effects
@@
 			)
 		)
-		(property "Footprint" ""
+		(property "Footprint" "B3F_1000:B3F1002"
 			(at 193.04 319.71 0)
 			(effects
@@
 			)
 		)
-		(property "Footprint" ""
+		(property "Footprint" "B3F_1000:B3F1002"
 			(at 107.95 299.39 0)
 			(effects
@@
 			)
 		)
-		(property "Footprint" ""
+		(property "Footprint" "B3F_1000:B3F1002"
 			(at 193.04 135.56 0)
 			(effects
@@
 			)
 		)
-		(property "Footprint" ""
+		(property "Footprint" "B3F_1000:B3F1002"
 			(at 193.04 299.39 0)
 			(effects
@@
 			)
 		)
-		(property "Footprint" ""
+		(property "Footprint" "B3F_1000:B3F1002"
 			(at 78.74 196.52 0)
 			(effects
@@
 			)
 		)
-		(property "Footprint" ""
+		(property "Footprint" "B3F_1000:B3F1002"
 			(at 107.95 319.71 0)
 			(effects
@@
 			)
 		)
-		(property "Footprint" ""
+		(property "Footprint" "B3F_1000:B3F1002"
 			(at 165.1 196.52 0)
 			(effects
@@
 			)
 		)
-		(property "Footprint" ""
+		(property "Footprint" "B3F_1000:B3F1002"
 			(at 193.04 216.84 0)
 			(effects
@@
 			)
 		)
-		(property "Footprint" ""
+		(property "Footprint" "B3F_1000:B3F1002"
 			(at 107.95 216.84 0)
 			(effects
@@
 			)
 		)
-		(property "Footprint" ""
+		(property "Footprint" "B3F_1000:B3F1002"
 			(at 107.95 155.88 0)
 			(effects
@@
 			)
 		)
-		(property "Footprint" ""
+		(property "Footprint" "B3F_1000:B3F1002"
 			(at 193.04 196.52 0)
 			(effects
@@
 			)
 		)
-		(property "Footprint" ""
+		(property "Footprint" "B3F_1000:B3F1002"
 			(at 165.1 135.56 0)
 			(effects
@@
 			)
 		)
-		(property "Footprint" ""
+		(property "Footprint" "B3F_1000:B3F1002"
 			(at 78.74 299.39 0)
 			(effects
@@
 			)
 		)
-		(property "Footprint" ""
+		(property "Footprint" "B3F_1000:B3F1002"
 			(at 165.1 319.71 0)
 			(effects
@@
 			)
 		)
-		(property "Footprint" ""
+		(property "Footprint" "B3F_1000:B3F1002"
 			(at 107.95 196.52 0)
 			(effects
